Commit message: new commit

File: src/Universal_Robots_ROS2_Description/urdf/ur5_macro.xacro (robot description, xacro)
@@ -3,5 +3,4 @@
   <xacro:macro name="ur5" params="prefix">
     <!-- create link fixed to the "world" -->
-    <link name="${prefix}world"/>
     <!-- links -  main serial chain -->
     <link name="${prefix}base_link"/>
@@ -140,9 +139,9 @@
     </link>
     <!-- base_joint fixes base_link to the environment -->
-    <joint name="${prefix}base_joint" type="fixed">
+    <!--<joint name="${prefix}base_joint" type="fixed">
       <origin rpy="0 0 0" xyz="0 0 0"/>
       <parent link="${prefix}world"/>
       <child link="${prefix}base_link"/>
-    </joint>
+    </joint> -->
     <!-- joints - main serial chain -->
     <joint name="${prefix}base_link-base_link_inertia" type="fixed">

File: src/my_robot_description/urdf/ur5.xacro (robot description, xacro)
@@ -1,12 +1,119 @@
 <?xml version="1.0"?>
 <robot name="leo" xmlns:xacro="http://ros.org/wiki/xacro">
+  <!-- Root link expected by UR macro -->
+  <link name="world"/>
+  <link name="robot1_world"/>
   <!-- Include Robot Macros -->
   <xacro:include filename="$(find ur_description)/urdf/ur5_macro.xacro"/>
   <xacro:include
     filename="$(find my_robot_moveit_config)/config/ros2_control_ignition.xacro"/>
+  <!-- Spawn UR5 -->
   <xacro:ur5 prefix="robot1_"/>
-   <xacro:leo_ros2_control_ignition
+   <!-- World placement joints -->
+  <joint name="robot1_world_to_world" type="fixed">
+    <parent link="world"/>
+    <child link="robot1_world"/>
+    <origin xyz="0 0 0" rpy="0 0 0"/>
+  </joint>
+  <joint name="robot1_joint_to_world" type="fixed">
+    <parent link="robot1_world"/>
+    <child link="robot1_base_link"/>
+    <origin xyz="0 0 0.80" rpy="0 0 0"/>
+  </joint>
+  <link name="table">
+        <visual>
+            <origin xyz="0 0 0" rpy="0 0 0"/>
+            <geometry>
+                <box size="1.0 1.0 0.75"/>
+            </geometry>
+            <material name="Grey">
+                <color rgba="0.7 0.7 0.7 1.0"/>
+            </material>
+        </visual>
+        <collision>
+            <origin xyz="0 0 0" rpy="0 0 0"/>
+            <geometry>
+                <box size="1.0 1.0 0.75"/>
+            </geometry>
+        </collision>
+        <inertial>
+            <mass value="500"/>
+            <origin xyz="0 0 0" rpy="0 0 0"/>
+            <inertia ixx="0.001" ixy="0" ixz="0" iyy="0.001" iyz="0" izz="0.001"/>
+        </inertial>
+    </link>
+    <gazebo reference="table">
+        <material>Gazebo/Black</material>
+        <!-- <transparency>1.0</transparency> -->
+    </gazebo>
+    <joint name="table_to_world" type="fixed">
+        <parent link="world"/>
+        <child link="table"/>
+        <origin xyz="0.0 0.6 0.375" rpy="0.0 0.0 0.0"/>
+    </joint>
+  <link name="camera">
+    <visual>
+      <geometry>
+        <box size="0.05 0.05 0.05" />
+      </geometry>
+      <material name="blue">
+        <color rgba="0.0 0.0 1.0 1.0"/>
+      </material>
+    </visual>
+    <collision>
+      <geometry>
+        <box size="0.1 0.1 0.1" />
+      </geometry>
+    </collision>
+    <inertial>
+      <mass value="0.1"/>
+      <origin xyz="0.0 0.0 0.0" rpy="0.0 0.0 0.0"/>
+      <inertia ixx="0.000166667" ixy="0.0" ixz="0.0" iyy="0.000166667" iyz="0.0" izz="0.000166667"/>
+    </inertial>
+  </link>
+  <joint name="world_to_camera" type="fixed">
+    <parent link="world"/>
+    <child link="camera"/>
+    <origin xyz="0.0 0.6 1.75" rpy="0.0 ${pi/2} 0.0"/>
+  </joint>
+  <gazebo reference="camera">
+    <sensor name="camera" type="camera">
+      <camera>
+        <camera_info_topic>camera/camera_info</camera_info_topic>
+        <horizontal_fov>1.047</horizontal_fov>
+        <image>
+          <width>320</width>
+          <height>240</height>
+        </image>
+        <clip>
+          <near>0.1</near>
+          <far>100</far>
+        </clip>
+      </camera>
+      <always_on>1</always_on>
+      <update_rate>30</update_rate>
+      <visualize>true</visualize>
+      <topic>camera/image_raw</topic>
+    </sensor>
+    <!--<sensor name="depth_camera1" type="depth_camera">
+          <update_rate>10</update_rate>
+          <topic>depth_camera</topic>
+          <camera>
+            <horizontal_fov>1.05</horizontal_fov>
+            <image>
+              <width>256</width>
+              <height>256</height>
+              <format>R_FLOAT32</format>
+            </image>
+            <clip>
+              <near>0.1</near>
+              <far>10.0</far>
+            </clip>
+          </camera>
+          </sensor> -->
+  </gazebo>
+  <!-- ros2_control -->
+  <xacro:leo_ros2_control_ignition
     name="Robot1System"
     initial_positions_file="$(find my_robot_moveit_config)/config/initial_positions.yaml"/>
-  <!-- Tables and camera can be included here, omitted for brevity -->
 </robot>

File: src/my_robot_moveit_config/config/ros2_control_ignition.xacro (robot description, xacro)
@@ -9,5 +9,5 @@
     <ros2_control name="${name}" type="system">
       <hardware>
-        <plugin>gz_ros2_control/GazeboSystem</plugin>
+         <plugin>gz_ros2_control/GazeboSimSystem</plugin>
       </hardware>
       <joint name="robot1_shoulder_pan_joint">
